Commit message: changed paths of urdf to relative

File: unitree_g1/models/urdf/g1_29dof_with_hand_rev_1_0.urdf (robot description, URDF)
Before this commit: robot g1_29dof_with_hand_rev_1_0, 63 links, 62 joints
Links:
- link L_hand_base_link: geometry collision mesh filename=meshes/L_hand_base_link.STL; visual mesh filename=meshes/L_hand_base_link.STL
- link L_index_distal: geometry collision mesh filename=meshes/L_index_distal.STL; visual mesh filename=meshes/L_index_distal.STL
- link L_index_proximal: geometry collision mesh filename=meshes/L_index_proximal.STL; visual mesh filename=meshes/L_index_proximal.STL
- link L_middle_distal: geometry collision mesh filename=meshes/L_middle_distal.STL; visual mesh filename=meshes/L_middle_distal.STL
- link L_middle_proximal: geometry collision mesh filename=meshes/L_middle_proximal.STL; visual mesh filename=meshes/L_middle_proximal.STL
- link L_pinky_distal: geometry collision mesh filename=meshes/L_pinky_distal.STL; visual mesh filename=meshes/L_pinky_distal.STL
- link L_pinky_proximal: geometry collision mesh filename=meshes/L_pinky_proximal.STL; visual mesh filename=meshes/L_pinky_proximal.STL
- link L_ring_distal: geometry collision mesh filename=meshes/L_ring_distal.STL; visual mesh filename=meshes/L_ring_distal.STL
- link L_ring_proximal: geometry collision mesh filename=meshes/L_ring_proximal.STL; visual mesh filename=meshes/L_ring_proximal.STL
- link L_thumb_distal: geometry collision mesh filename=meshes/L_thumb_distal.STL; visual mesh filename=meshes/L_thumb_distal.STL
- link L_thumb_intermediate: geometry collision mesh filename=meshes/L_thumb_intermediate.STL; visual mesh filename=meshes/L_thumb_intermediate.STL
- link L_thumb_proximal: geometry collision mesh filename=meshes/L_thumb_proximal.STL; visual mesh filename=meshes/L_thumb_proximal.STL
- link L_thumb_proximal_base: geometry collision mesh filename=meshes/L_thumb_proximal_base.STL; visual mesh filename=meshes/L_thumb_proximal_base.STL
- link R_hand_base_link: geometry collision mesh filename=meshes/R_hand_base_link.STL; visual mesh filename=meshes/R_hand_base_link.STL
- link R_index_distal: geometry collision mesh filename=meshes/R_index_distal.STL; visual mesh filename=meshes/R_index_distal.STL
- link R_index_proximal: geometry collision mesh filename=meshes/R_index_proximal.STL; visual mesh filename=meshes/R_index_proximal.STL
- link R_middle_distal: geometry collision mesh filename=meshes/R_middle_distal.STL; visual mesh filename=meshes/R_middle_distal.STL
- link R_middle_proximal: geometry collision mesh filename=meshes/R_middle_proximal.STL; visual mesh filename=meshes/R_middle_proximal.STL
- link R_pinky_distal: geometry collision mesh filename=meshes/R_pinky_distal.STL; visual mesh filename=meshes/R_pinky_distal.STL
- link R_pinky_proximal: geometry collision mesh filename=meshes/R_pinky_proximal.STL; visual mesh filename=meshes/R_pinky_proximal.STL
- link R_ring_distal: geometry collision mesh filename=meshes/R_ring_distal.STL; visual mesh filename=meshes/R_ring_distal.STL
- link R_ring_proximal: geometry collision mesh filename=meshes/R_ring_proximal.STL; visual mesh filename=meshes/R_ring_proximal.STL
- link R_thumb_distal: geometry collision mesh filename=meshes/R_thumb_distal.STL; visual mesh filename=meshes/R_thumb_distal.STL
- link R_thumb_intermediate: geometry collision mesh filename=meshes/R_thumb_intermediate.STL; visual mesh filename=meshes/R_thumb_intermediate.STL
- link R_thumb_proximal: geometry collision mesh filename=meshes/R_thumb_proximal.STL; visual mesh filename=meshes/R_thumb_proximal.STL
- link R_thumb_proximal_base: geometry collision mesh filename=meshes/R_thumb_proximal_base.STL; visual mesh filename=meshes/R_thumb_proximal_base.STL
- link head_link: geometry collision mesh filename=meshes/head_link.STL; visual mesh filename=meshes/head_link.STL
- link left_ankle_pitch_link: geometry collision mesh filename=meshes/left_ankle_pitch_link.STL; visual mesh filename=meshes/left_ankle_pitch_link.STL
- link left_ankle_roll_link: geometry collision sphere radius=0.005; collision sphere radius=0.005
- link left_elbow_link: geometry collision mesh filename=meshes/left_elbow_link.STL; visual mesh filename=meshes/left_elbow_link.STL
- link left_hip_pitch_link: geometry collision mesh filename=meshes/left_hip_pitch_link.STL; visual mesh filename=meshes/left_hip_pitch_link.STL
- link left_hip_roll_link: geometry collision mesh filename=meshes/left_hip_roll_link.STL; visual mesh filename=meshes/left_hip_roll_link.STL
- link left_hip_yaw_link: geometry collision mesh filename=meshes/left_hip_yaw_link.STL; visual mesh filename=meshes/left_hip_yaw_link.STL
- link left_knee_link: geometry collision mesh filename=meshes/left_knee_link.STL; visual mesh filename=meshes/left_knee_link.STL
- link left_shoulder_pitch_link: geometry collision cylinder length=0.05 radius=0.03; visual mesh filename=meshes/left_shoulder_pitch_link.STL
- link left_shoulder_roll_link: geometry collision cylinder length=0.03 radius=0.03; visual mesh filename=meshes/left_shoulder_roll_link.STL
- link left_shoulder_yaw_link: geometry collision mesh filename=meshes/left_shoulder_yaw_link.STL; visual mesh filename=meshes/left_shoulder_yaw_link.STL
- link left_wrist_pitch_link: geometry collision mesh filename=meshes/left_wrist_pitch_link.STL; visual mesh filename=meshes/left_wrist_pitch_link.STL
- link left_wrist_roll_link: geometry collision mesh filename=meshes/left_wrist_roll_link.STL; visual mesh filename=meshes/left_wrist_roll_link.STL
- link left_wrist_yaw_link: geometry collision mesh filename=meshes/left_wrist_yaw_link.STL; visual mesh filename=meshes/left_wrist_yaw_link.STL
- link logo_link: geometry collision mesh filename=meshes/logo_link.STL; visual mesh filename=meshes/logo_link.STL
- link pelvis: geometry visual mesh filename=meshes/pelvis.STL
- link pelvis_contour_link: geometry collision mesh filename=meshes/pelvis_contour_link.STL; visual mesh filename=meshes/pelvis_contour_link.STL
- link right_ankle_pitch_link: geometry collision mesh filename=meshes/right_ankle_pitch_link.STL; visual mesh filename=meshes/right_ankle_pitch_link.STL
- link right_ankle_roll_link: geometry collision sphere radius=0.005; collision sphere radius=0.005
- link right_elbow_link: geometry collision mesh filename=meshes/right_elbow_link.STL; visual mesh filename=meshes/right_elbow_link.STL
- link right_hip_pitch_link: geometry collision mesh filename=meshes/right_hip_pitch_link.STL; visual mesh filename=meshes/right_hip_pitch_link.STL
- link right_hip_roll_link: geometry collision mesh filename=meshes/right_hip_roll_link.STL; visual mesh filename=meshes/right_hip_roll_link.STL
- link right_hip_yaw_link: geometry collision mesh filename=meshes/right_hip_yaw_link.STL; visual mesh filename=meshes/right_hip_yaw_link.STL
- link right_knee_link: geometry collision mesh filename=meshes/right_knee_link.STL; visual mesh filename=meshes/right_knee_link.STL
- link right_shoulder_pitch_link: geometry collision cylinder length=0.05 radius=0.03; visual mesh filename=meshes/right_shoulder_pitch_link.STL
- link right_shoulder_roll_link: geometry collision cylinder length=0.03 radius=0.03; visual mesh filename=meshes/right_shoulder_roll_link.STL
- link right_shoulder_yaw_link: geometry collision mesh filename=meshes/right_shoulder_yaw_link.STL; visual mesh filename=meshes/right_shoulder_yaw_link.STL
- link right_wrist_pitch_link: geometry collision mesh filename=meshes/right_wrist_pitch_link.STL; visual mesh filename=meshes/right_wrist_pitch_link.STL
- link right_wrist_roll_link: geometry collision mesh filename=meshes/right_wrist_roll_link.STL; visual mesh filename=meshes/right_wrist_roll_link.STL
- link right_wrist_yaw_link: geometry collision mesh filename=meshes/right_wrist_yaw_link.STL; visual mesh filename=meshes/right_wrist_yaw_link.STL
- link torso_link: geometry collision mesh filename=meshes/torso_link_rev_1_0.STL; visual mesh filename=meshes/torso_link_rev_1_0.STL
- link waist_roll_link: geometry visual mesh filename=meshes/waist_roll_link_rev_1_0.STL
- link waist_yaw_link: geometry visual mesh filename=meshes/waist_yaw_link_rev_1_0.STL
